File: LM399VoltageStandard.kicad_sch (KiCad schematic)
At the start: 27 parts, among them U1 LM399, U2 LT1001

Commit message: Power Supply
Parts:
- added C10, C11, C17, C19, C6, C7, C8: 100n, Capacitor_SMD:C_0603_1608Metric, symbol Device:C_Small
- added C12, C13: 100n, Capacitor_SMD:C_0805_2012Metric, symbol Device:C_Small
- added C14, C18, C9: 47u, Capacitor_THT:CP_Radial_D5.0mm_P2.00mm, symbol Device:C_Polarized_Small_US
- added C15, C16, C4, C5: 1000u, Capacitor_THT:CP_Radial_D10.0mm_P3.80mm, symbol Device:C_Polarized_Small_US
- added D1, D2, D3, D4: AU3PG-M3/87A, Package_TO_SOT_SMD:TO-277A, symbol Device:D
- added D5: 1N4148, Diode_THT:D_DO-35_SOD27_P7.62mm_Horizontal, symbol Diode:1N4148
- added D6: KBP10, Diode_THT:Diode_Bridge_19.0x3.5x10.0mm_P5.0mm, symbol Diode_Bridge:B380C2300-1500A
- added J1: Screw_Terminal_01x04, TerminalBlock:TerminalBlock_MaiXu_MX126-5.0-04P_1x04_P5.00mm, symbol Connector:Screw_Terminal_01x04
- added R2: 250, Resistor_SMD:R_0603_1608Metric, symbol Device:R
- added R3: 150k, Resistor_SMD:R_0603_1608Metric, symbol Device:R
- added U3: LT3045xDD, Package_DFN_QFN:DFN-10-1EP_3x3mm_P0.5mm_EP1.65x2.38mm, symbol Regulator_Linear:LT3045xDD
- added U4: 7818, symbol Regulator_Linear:L7818
- added U5: LM7815, Package_TO_SOT_THT:TO-220-3_Vertical, symbol Regulator_Linear:LM7815_TO220
- C1, C2: footprint (none) -> Capacitor_SMD:C_0603_1608Metric
- U1: Link (none) -> https://allegro.pl/oferta/lm399h-to46-4-uklad-scalony-11313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
Connections:
- net +15V: now also C10.1, C6.1, C9.1, U3.10 (OUT), U3.9 (OUTS)
- net +15V_H: now also C13.1, C14.1, D5.1 (K), U5.3 (VO)
- net Masa: now also C10.2, C11.2, C12.2, C13.2, C14.2, C15.2, C16.2, C17.2, C18.2, C19.2, C4.2, C5.2, C6.2, C7.2, C8.2, C9.2, D1.1 (A), D1.2 (A), D2.1 (A), D2.2 (A), D5.2 (A), D6.1 (-), R2.2, R3.2, U3.11 (GND), U3.8 (GND), U4.2 (GND), U5.2 (GND)
- new net: C12.1, C15.1, C16.1, D6.4 (+), U5.1 (VI)
- new net: C4.1, C5.1, C7.1, C8.1, D3.3 (K), D4.3 (K), U4.1 (IN)
- new net: D2.3 (K), D3.1 (A), D3.2 (A), J1.3 (Pin_3)
- new net: R2.1, U3.5 (ILIM)
- new net: C11.1, R3.1, U3.7 (SET)
- new net: C17.1, C18.1, C19.1, U3.1 (IN), U3.2 (IN), U3.3 (EN/UV), U3.6 (PGFB), U4.3 (OUT)
- new net: D1.3 (K), D4.1 (A), D4.2 (A), J1.4 (Pin_4)
- new net: D6.3, J1.1 (Pin_1)
- new net: D6.2, J1.2 (Pin_2)
- no-connect marks 3 -> 4
Other:
- note added: "DP-241-4-20"
- moved on the sheet: C1, C3, R1, R10, R11, R12, R13, R14, R15, R16, R17, R18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

Commit message: Started PCB
Parts:
- removed C3: 10n, symbol Device:C_Small
- removed D5: 1N4148, Diode_THT:D_DO-35_SOD27_P7.62mm_Horizontal, symbol Diode:1N4148
- removed JP2, JP3, JP4, JP5, JP6, JP7: Jumper_2_Open, symbol Jumper:Jumper_2_Open
- removed R18, R19: 8M25, symbol Device:R
- added C20: 100n, Capacitor_SMD:C_0603_1608Metric, symbol Device:C_Small
- added C21: 1n, Capacitor_SMD:C_0603_1608Metric, symbol Device:C_Small
- added C22: 10u, Capacitor_Tantalum_SMD:CP_EIA-7132-20_AVX-U, symbol Device:C_Polarized_Small_US
- added JP10, JP11, JP12, JP13, JP14, JP8, JP9: Jumper_2_Open, Jumper:SolderJumper-2_P1.3mm_Open_RoundedPad1.0x1.5mm, symbol Jumper:Jumper_2_Open
- added R6: 2k, Resistor_SMD:R_1206_3216Metric, symbol Device:R
- R1, R13: footprint (none) -> Resistor_SMD:R_0603_1608Metric
- R10, R14: footprint (none) -> Resistor_THT:R_Axial_DIN0204_L3.6mm_D1.6mm_P7.62mm_Horizontal
- R11: footprint (none) -> Resistor_SMD:R_0603_1608Metric; Link (none) -> https://www.mouser.pl/ProductDetail/TE-Connectivity-Holswor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
- R12: value 0R -> 8M25; footprint (none) -> Resistor_THT:R_Axial_DIN0204_L3.6mm_D1.6mm_P7.62mm_Horizontal; Link (none) -> https://www.mouser.pl/ProductDetail/Xicon/270-8.25M-RC?qs=s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; now fitted
- R15: value 8M25 -> 32M; footprint (none) -> Resistor_THT:R_Axial_DIN0207_L6.3mm_D2.5mm_P10.16mm_Horizontal; Link https://www.mouser.pl/ProductDetail/Xicon/270-8.25M-RC?qs=s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 -> https://www.mouser.pl/ProductDetail/Vishay-Dale/CMF554M1200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
- R16: value 8M25 -> 32M; footprint (none) -> Resistor_SMD:R_0805_2012Metric; Link https://www.mouser.pl/ProductDetail/Xicon/270-8.25M-RC?qs=s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 -> https://www.mouser.pl/ProductDetail/Kamaya/RGC1-10C2054FTP?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; now not fitted
- R17: value 8M25 -> 50R; footprint (none) -> Resistor_SMD:R_0805_2012Metric; Link https://www.mouser.pl/ProductDetail/Xicon/270-8.25M-RC?qs=s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 -> https://www.mouser.pl/ProductDetail/YAGEO/RT0805BRD071M02L?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
- R4: footprint (none) -> LM399VoltageStandard:ZFoilResistor; Link (none) -> https://www.mouser.pl/ProductDetail/Vishay-Precision-Group-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
- R5: footprint (none) -> Resistor_THT:R_Axial_DIN0207_L6.3mm_D2.5mm_P10.16mm_Horizontal; Link (none) -> https://www.mouser.pl/ProductDetail/Vishay-Precision-Group-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
- R7, R8: footprint (none) -> Resistor_SMD:R_0805_2012Metric
- R9: footprint (none) -> Resistor_THT:R_Axial_DIN0207_L6.3mm_D2.5mm_P10.16mm_Horizontal
- U4: footprint (none) -> Package_TO_SOT_SMD:TO-263-2; Link (none) -> https://www.mouser.pl/ProductDetail/onsemi/MC7818CD2TR4G?qs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
Connections:
- net 10V: now also R17.2, C20.1, C22.1; no longer R11.1, R12.1, R4.1, U2.6
- net Masa: now also C20.2, C21.2, C22.2; no longer C12.2, C13.2, C14.2, C15.2, C16.2, D6.1 (-), U1.4, U5.2 (GND)
- net at R13.1: now also JP8.1 (A); no longer R12.2
- net at R10.2, R11.2, R13.2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: now also R15.2, R16.2
- net at R7.1: now also JP9.1 (A)
- net at R1.2, U1.1, U2.3 (+): now also C21.1
- net at R8.1: now also JP10.1 (A)
- net at R10.1: now also JP12.1 (A)
- net at R16.1: now also R15.1, JP14.1 (A)
- net at R9.1: now also JP11.1 (A)
- net at R14.1: now also R12.2; no longer R15.2
- net at R17.1: now also R4.1, U2.6, JP10.2 (B), JP11.2 (B), JP12.2 (B), JP13.2 (B), JP14.2 (B), JP8.2 (B), JP9.2 (B), R6.1; no longer R16.2
- new net: JP13.1 (A), R12.1
- new net: R11.1, R6.2
- new net GND_H: C12.2, C13.2, C14.2, C15.2, C16.2, D6.1 (-), U1.4, U5.2 (GND)
Other:
- note added: "4k385 total"
- moved on the sheet: C12, C13, C14, C15, C16, D6, R11, R13, R4, R5, U5
