File: LM399VoltageStandard.kicad_sch (KiCad schematic)
At the start: 45 parts, among them U1 LM399, U2 LT1001

Commit message: Final Version
Parts:
- removed H5, H6, H7, H8: MountingHole, MountingHole:MountingHole_3.2mm_M3_DIN965_Pad, symbol Mechanical:MountingHole
- added C46: 100n, Capacitor_SMD:C_0603_1608Metric, symbol Device:C_Small
- added H5, H6, H7, H8: MountingHole_Pad, MountingHole:MountingHole_3.2mm_M3_Pad_TopBottom, symbol Mechanical:MountingHole_Pad
- added JP15, JP16, JP17, JP18: Jumper_2_Open, Jumper:SolderJumper-2_P1.3mm_Open_RoundedPad1.0x1.5mm, symbol Jumper:Jumper_2_Open
- added U12: LM35-LP, Package_TO_SOT_THT:TO-92_Inline, symbol Sensor_Temperature:LM35-LP
Connections:
- net +15V_H: now also C46.1, U12.1 (+V_{S})
- net Masa: now also C46.2, JP15.2 (B), JP16.2 (B), JP17.2 (B), JP18.2 (B), U12.3 (GND)
- new net: H5.1, JP15.1 (A)
- new net: H6.1, JP16.1 (A)
- new net: H7.1, JP17.1 (A)
- new net: H8.1, JP18.1 (A)
- new net TEMP_SENSE: U12.2 (V_{OUT})
