File: MCU.kicad_sch (KiCad schematic)
At the start: 5 parts, among them U7 STM32G431C6Tx

Commit message: Final Version
Parts:
- added C33, C36, C37, C40, C41, C43, C47: 100n, Capacitor_SMD:C_0603_1608Metric, symbol Device:C_Small
- added C34, C35: 14p, Capacitor_SMD:C_0603_1608Metric, symbol Device:C_Small
- added C38: 10u, Capacitor_SMD:C_0805_2012Metric, symbol Device:C_Small
- added C39: 2u2, Capacitor_SMD:C_0603_1608Metric, symbol Device:C_Small
- added D5: LED_BGKR, LED_THT:LED_D5.0mm-4_RGB_Wide_Pins, symbol Device:LED_BGKR
- added FB1: 120R, Inductor_SMD:L_0603_1608Metric, symbol Device:FerriteBead_Small
- added J2: USB_B_Micro, Connector_USB:USB_Micro-B_Technik_TWP-4002D-H3, symbol Connector:USB_B_Micro
- added J3: Conn_01x04, Connector_PinHeader_2.54mm:PinHeader_1x04_P2.54mm_Vertical, symbol Connector_Generic:Conn_01x04
- added J4: Conn_01x02, Connector_PinHeader_2.54mm:PinHeader_1x02_P2.54mm_Vertical, symbol Connector_Generic:Conn_01x02
- added R18, R19: 10k, Resistor_SMD:R_0603_1608Metric, symbol Device:R
- added R20: 1k5, Resistor_SMD:R_0603_1608Metric, symbol Device:R
- added R21, R22: 4k7, Resistor_SMD:R_0603_1608Metric, symbol Device:R
- added R28: 100R, Resistor_SMD:R_0603_1608Metric, symbol Device:R
- added U10: TMP102xxDRL, Package_TO_SOT_SMD:SOT-563, symbol Sensor_Temperature:TMP102xxDRL
- added U8: USBLC6-2SC6, Package_TO_SOT_SMD:SOT-23-6, symbol Power_Protection:USBLC6-2SC6
- added U9: FM24C64B, Package_SO:SOIC-8_3.9x4.9mm_P1.27mm, symbol Memory_NVRAM:FM24C64B
- added Y1: Crystal_GND24, Crystal:Crystal_SMD_EuroQuartz_X22-4Pin_2.5x2.0mm_HandSoldering, symbol Device:Crystal_GND24
Connections:
- net +3V3: now also C36.1, C37.1, C38.1, C40.1, C41.1, FB1.2, J3.1 (Pin_1), R20.1, R21.1, R22.1, U10.5 (V+), U9.8 (VDD); no longer C32.1, U7.21 (VDDA)
- net Masa: now also C33.2, C34.2, C35.2, C36.2, C37.2, C38.2, C39.2, C40.2, C41.2, C43.2, C47.2, D5.3 (K), J2.5 (GND), J3.4 (Pin_4), J4.2 (Pin_2), R19.2, U10.2 (GND), U10.4 (ADD0), U8.2 (GND), U9.1 (A0), U9.2 (A1), U9.3 (A2), U9.4 (VSS), U9.7 (WP), Y1.2 (G), Y1.4 (G)
- net RCC_OSC_IN: now also C34.1, Y1.3
- net RCC_OSC_OUT: now also C35.1, Y1.1
- net SYS_JTCK_SWCLK: now also J3.3 (Pin_3)
- net SYS_JTMS_SWDIO: now also J3.2 (Pin_2)
- net USB_D+: now also R20.2, U8.4 (I/O2)
- net USB_D-: now also U8.6 (I/O1)
- net REFERENCE_VOLTAGE_SENSE: now reaches U7.11 (PA3)
- net CAL_EN: now reaches U7.12 (PA4)
- net CAL_EN: now also J4.1 (Pin_1)
- net LED_R: now reaches U7.13 (PA5)
- net LED_R: now also D5.4 (RA)
- net LED_G: now reaches U7.14 (PA6)
- net LED_G: now also D5.2 (GA)
- net LED_B: now reaches U7.15 (PA7)
- net LED_B: now also D5.1 (BA)
- net HEATER_SENSE_OUT: now reaches U7.16 (PB0)
- net HEATER_SENSE_OUT: now also C43.1
- net HEATER_VOLTAGE_SENSE: now reaches U7.17 (PB1)
- net at U7.20 (VREF+): now also C32.1, U7.21 (VDDA), C33.1, C39.1, FB1.1
- net at U7.26 (PB12): now also C47.1, R28.2
- net VBUS_SENSE: now reaches U7.32 (PA10)
- net VBUS_SENSE: now also R18.2, R19.1
- net SCL1: now reaches U7.39 (PA15)
- net SCL1: now also R22.2, U10.1 (SCL), U9.6 (SCL)
- net SDA1: now reaches U7.44 (PB7)
- net SDA1: now also R21.2, U10.6 (SDA), U9.5 (SDA)
- new net D+: J2.3 (D+), U8.3 (I/O2)
- new net D-: J2.2 (D-), U8.1 (I/O1)
- new net TEMP_SENSE: R28.1
- new net Vbus: J2.1 (VBUS), R18.1, U8.5 (VBUS)
- no-connect marks 0 -> 3
Other:
- note added: "Crystal"
- note added: "EEPROM"
- note added: "USB Connector"
- moved on the sheet: C29, C30, C31, C32, U7

Commit message: Added BOM
Parts:
- C38: Price (none) -> 1,51zł
- C39, FB1: Price (none) -> 0,36zł
- D5: Price (none) -> 0,97zł
- U10: Price (none) -> 4,15zł
- U7: Price (none) -> 16,72zł
- U8: Price (none) -> 1,59zł
- U9: Price (none) -> 1,12zł
- Y1: Price (none) -> 0,87zł
