File: PowerSupply.kicad_sch (KiCad schematic)
At the start: 41 parts, among them J1 Screw_Terminal_01x02, U11 INA180B3, U3 LT3045xDD, U4 TLV75533PDRV, U5 LM7815, U6 LM7805_TO220

Commit message: Changed Diodes in rectifier
Parts:
- D1, D2, D3, D4: value AU3PG-M3/87A -> PUUP3JH; Link https://www.mouser.pl/ProductDetail/Vishay-Semiconductors/A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 -> https://www.mouser.pl/en/ProductDetail/Taiwan-Semiconductor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
Changed lines of the file:
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@@
 			)
 		)
-		(property "Value" "AU3PG-M3/87A"
+		(property "Value" "PUUP3JH"
 			(at 63.246 23.368 0)
 			(hide yes)
@@
 			)
 		)
-		(property "Link" "https://www.mouser.pl/ProductDetail/Vishay-Semiconductors/AU3PG-M3-87A?qs=z5NHsHGj0DHMjKPjFfMplA%3D%3D&mgh=1&vip=1&utm_id=20549636368&utm_source=google&utm_medium=cpc&utm_marketing_tactic=emeacorp&gad_source=1&gad_campaignid=20549637556&gclid=Cj0KCQjwjb3SBhDgARIsAMKiWzh7-kt-LDRCP2d-i5VUVBCPEHf-Q3h3HIx2QY1Ba2Nftnte4OfJRv0aAoGjEALw_wcB"
+		(property "Link" "https://www.mouser.pl/en/ProductDetail/Taiwan-Semiconductor/PUUP3JH?qs=NeOn4crkEuub6tf3VFnloQ%3D%3D"
 			(at 58.42 29.21 0)
 			(hide yes)
@@
 			)
 		)
-		(property "Value" "AU3PG-M3/87A"
+		(property "Value" "PUUP3JH"
 			(at 46.736 25.654 0)
 			(show_name no)
@@
 			)
 		)
-		(property "Link" "https://www.mouser.pl/ProductDetail/Vishay-Semiconductors/AU3PG-M3-87A?qs=z5NHsHGj0DHMjKPjFfMplA%3D%3D&mgh=1&vip=1&utm_id=20549636368&utm_source=google&utm_medium=cpc&utm_marketing_tactic=emeacorp&gad_source=1&gad_campaignid=20549637556&gclid=Cj0KCQjwjb3SBhDgARIsAMKiWzh7-kt-LDRCP2d-i5VUVBCPEHf-Q3h3HIx2QY1Ba2Nftnte4OfJRv0aAoGjEALw_wcB"
+		(property "Link" "https://www.mouser.pl/en/ProductDetail/Taiwan-Semiconductor/PUUP3JH?qs=NeOn4crkEuub6tf3VFnloQ%3D%3D"
 			(at 58.42 44.45 0)
 			(hide yes)
@@
 			)
 		)
-		(property "Value" "AU3PG-M3/87A"
+		(property "Value" "PUUP3JH"
 			(at 60.198 32.004 0)
 			(hide yes)
@@
 			)
 		)
-		(property "Link" "https://www.mouser.pl/ProductDetail/Vishay-Semiconductors/AU3PG-M3-87A?qs=z5NHsHGj0DHMjKPjFfMplA%3D%3D&mgh=1&vip=1&utm_id=20549636368&utm_source=google&utm_medium=cpc&utm_marketing_tactic=emeacorp&gad_source=1&gad_campaignid=20549637556&gclid=Cj0KCQjwjb3SBhDgARIsAMKiWzh7-kt-LDRCP2d-i5VUVBCPEHf-Q3h3HIx2QY1Ba2Nftnte4OfJRv0aAoGjEALw_wcB"
+		(property "Link" "https://www.mouser.pl/en/ProductDetail/Taiwan-Semiconductor/PUUP3JH?qs=NeOn4crkEuub6tf3VFnloQ%3D%3D"
 			(at 66.04 36.83 0)
 			(hide yes)
@@
 			)
 		)
-		(property "Value" "AU3PG-M3/87A"
+		(property "Value" "PUUP3JH"
 			(at 53.34 38.0999 90)
 			(hide yes)
@@
 			)
 		)
-		(property "Link" "https://www.mouser.pl/ProductDetail/Vishay-Semiconductors/AU3PG-M3-87A?qs=z5NHsHGj0DHMjKPjFfMplA%3D%3D&mgh=1&vip=1&utm_id=20549636368&utm_source=google&utm_medium=cpc&utm_marketing_tactic=emeacorp&gad_source=1&gad_campaignid=20549637556&gclid=Cj0KCQjwjb3SBhDgARIsAMKiWzh7-kt-LDRCP2d-i5VUVBCPEHf-Q3h3HIx2QY1Ba2Nftnte4OfJRv0aAoGjEALw_wcB"
+		(property "Link" "https://www.mouser.pl/en/ProductDetail/Taiwan-Semiconductor/PUUP3JH?qs=NeOn4crkEuub6tf3VFnloQ%3D%3D"
 			(at 50.8 36.83 0)
 			(hide yes)
