File: LM399VoltageStandard.kicad_pcb (KiCad board)
At the start: 4 copper layers, 100 x 100 mm, 123 parts, among them J1 Screw_Terminal_01x02, J2 USB_B_Micro, J3 Conn_01x04, J4 Conn_01x02, U1 LM399, U10 TMP102xxDRL, U11 INA180B3, U12 LM35-LP, U2 LT1001, U3 LT3045xDD, U4 TLV75533PDRV, U5 LM7815, U6 LM7805_TO220, U7 STM32G431C6Tx, U8 USBLC6-2SC6, U9 FM24C64B, Y1 Crystal_GND24

Commit message: Added BOM
Parts:
- C20: footprint Capacitor_SMD:C_0603_1608Metric -> Capacitor_SMD:C_1206_3216Metric
- moved C20 1.13 mm to (130.7, 49.3)
Changed lines of the file:
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@@
 		)
 	)
-	(footprint "Capacitor_SMD:C_0603_1608Metric"
+	(footprint "Capacitor_SMD:C_1206_3216Metric"
 		(layer "F.Cu")
-		(at 130.1325 48.325 -90)
-		(descr "Capacitor SMD 0603 (1608 Metric), square (rectangular) end terminal, IPC-7351 nominal, (Body size source: IPC-SM-782 page 76, https://www.pcb-3d.com/wordpress/wp-content/uploads/ipc-sm-782a_amendment_1_and_2.pdf)")
+		(at 130.7 49.3 -90)
+		(descr "Capacitor SMD 1206 (3216 Metric), square (rectangular) end terminal, IPC-7351 nominal, (Body size source: IPC-SM-782 page 76, https://www.pcb-3d.com/wordpress/wp-content/uploads/ipc-sm-782a_amendment_1_and_2.pdf)")
 		(tags "capacitor")
 		(property "Reference" "C20"
-			(at 0 -1.43 90)
+			(at 0 -1.85 270)
 			(layer "F.SilkS")
 			(effects
@@
 		)
 		(property "Value" "100n"
-			(at 0 1.43 90)
+			(at 0 1.85 270)
 			(layer "F.Fab")
 			(hide yes)
@@
 		)
 		(property "Datasheet" ""
-			(at 0 0 90)
+			(at 0 0 270)
 			(layer "F.Fab")
 			(hide yes)
@@
 		)
 		(property "Description" "Unpolarized capacitor, small symbol"
-			(at 0 0 90)
+			(at 0 0 270)
 			(layer "F.Fab")
 			(hide yes)
@@
 		)
 		(property "KiLib_Generator" "SMD_2terminal_chip_molded"
-			(at 0 0 90)
+			(at 0 0 270)
 			(layer "F.SilkS")
 			(hide yes)
@@
 			)
 		)
+		(property "Link" "https://www.mouser.pl/en/ProductDetail/Murata-Electronics/GRM3195C1H104JA05D?qs=sGAEpiMZZMvsSlwiRhF8qtsGU%2FCnaNeQltqslDj%252Bbfl9yz60Q4XpLA%3D%3D"
+			(at 0 0 270)
+			(unlocked yes)
+			(layer "F.Fab")
+			(hide yes)
+			(effects
+				(font
+					(size 1 1)
+					(thickness 0.15)
+				)
+			)
+		)
 		(property ki_fp_filters "C_*")
 		(sheetname "/")
@@
 		(duplicate_pad_numbers_are_jumpers no)
 		(fp_line
-			(start -0.14058 0.51)
-			(end 0.14058 0.51)
+			(start -0.711252 0.91)
+			(end 0.711252 0.91)
 			(stroke
 				(width 0.12)
@@
 		)
 		(fp_line
-			(start -0.14058 -0.51)
-			(end 0.14058 -0.51)
+			(start -0.711252 -0.91)
+			(end 0.711252 -0.91)
 			(stroke
 				(width 0.12)
@@
 		)
 		(fp_rect
-			(start -1.48 -0.73)
-			(end 1.48 0.73)
+			(start -2.3 -1.15)
+			(end 2.3 1.15)
 			(stroke
 				(width 0.05)
@@
 		)
 		(fp_rect
-			(start -0.8 -0.4)
-			(end 0.8 0.4)
+			(start -1.6 -0.8)
+			(end 1.6 0.8)
 			(stroke
 				(width 0.1)
@@
 		)
 		(fp_text user "${REFERENCE}"
-			(at 0 0 90)
+			(at 0 0 270)
 			(layer "F.Fab")
 			(effects
 				(font
-					(size 0.4 0.4)
-					(thickness 0.06)
+					(size 0.8 0.8)
+					(thickness 0.12)
 				)
 			)
 		)
 		(pad "1" smd roundrect
-			(at -0.775 0 270)
-			(size 0.9 0.95)
+			(at -1.475 0 270)
+			(size 1.15 1.8)
 			(layers "F.Cu" "F.Mask" "F.Paste")
-			(roundrect_rratio 0.25)
+			(roundrect_rratio 0.217391)
 			(net "/10V")
 			(pintype "passive")
 		)
 		(pad "2" smd roundrect
-			(at 0.775 0 270)
-			(size 0.9 0.95)
+			(at 1.475 0 270)
+			(size 1.15 1.8)
 			(layers "F.Cu" "F.Mask" "F.Paste")
-			(roundrect_rratio 0.25)
+			(roundrect_rratio 0.217391)
 			(net "Masa")
 			(pintype "passive")
 		)
 		(embedded_fonts no)
-		(model "${KICAD10_3DMODEL_DIR}/Capacitor_SMD.3dshapes/C_0603_1608Metric.step"
+		(model "${KICAD10_3DMODEL_DIR}/Capacitor_SMD.3dshapes/C_1206_3216Metric.step"
 			(offset
 				(xyz 0 0 0)
@@
 	)
 	(segment
+		(start 130.7 52.15)
+		(end 130.65 52.2)
+		(width 0.4)
+		(layer "F.Cu")
+		(net "Masa")
+	)
+	(segment
 		(start 82.6125 109)
 		(end 82.6125 108.9)
@@
 	)
 	(segment
-		(start 130.1325 49.1)
-		(end 130.1325 50.475)
-		(width 0.4)
-		(layer "F.Cu")
-		(net "Masa")
-	)
-	(segment
 		(start 121.2 115.4)
 		(end 122.55 115.4)
@@
 	)
 	(segment
+		(start 130.7 50.775)
+		(end 130.7 52.15)
+		(width 0.4)
+		(layer "F.Cu")
+		(net "Masa")
+	)
+	(segment
 		(start 77.15 120.8)
 		(end 77.15 119.65)
@@
 	)
 	(via
-		(at 130.1325 50.475)
+		(at 130.65 52.2)
 		(size 0.6)
 		(drill 0.3)

Commit message: Commit
Parts:
- removed C11: 100n, Capacitor_SMD:C_0603_1608Metric
- removed D1, D2, D3, D4: AU3PG-M3/87A, Package_TO_SOT_SMD:TO-277A
- removed R2: 250, Resistor_SMD:R_0603_1608Metric
- removed R3: 150k, Resistor_SMD:R_0603_1608Metric
- removed U3: LT3045xDD, Package_DFN_QFN:DFN-10-1EP_3x3mm_P0.5mm_EP1.65x2.38mm
- added C48: 1000u, Capacitor_THT:CP_Radial_D10.0mm_P3.80mm, F.Cu at (99.5, 110.8)
- added D6: B40C2300-1500A, Diode_THT:Diode_Bridge_19.0x3.5x10.0mm_P5.0mm, F.Cu at (110.5, 117.0)
- added U13: LM7815, Package_TO_SOT_THT:TO-220-3_Vertical, F.Cu at (112.0, 110.0)
- moved C19 8.70 mm to (112.2, 112.5)
- moved C9 7.52 mm to (122.5, 111.5), turned to 90 degrees
- moved C10 6.36 mm to (115.8, 112.5), turned to 180 degrees
Routing:
- net VIN: track 42.6 -> 91.4 mm, vias 2 -> 0
- net +15V: track 63.8 -> 73.5 mm, vias 4 -> 2
- net Net-(J1-Pin_2): track 17.1 -> 8.85 mm
- net Net-(J1-Pin_1): track 17.1 -> 8.85 mm
- net Net-(U3-SET): track 4.65 -> 0.00 mm
- net Net-(U3-ILIM): track 1.63 -> 0.00 mm
- net /MCU/USB_D+: track 7.96 -> 9.56 mm
- net Masa: track 113.7 -> 114.1 mm, vias 144 -> 133
