File: PCB/PowerSupply.kicad_sch (KiCad schematic)
At the start: 39 parts, among them J1 Screw_Terminal_01x02, U11 INA180B3, U13 LM7815, U4 TLV75533PDRV, U5 LM7815, U6 LM7805_TO220

Commit message: fixed BOM
Parts:
- removed D2, D3, D4: PUUP3JH, Package_TO_SOT_SMD:TO-277A, symbol Device:D
- added C45: 100n, Capacitor_SMD:C_0603_1608Metric, symbol Device:C_Small
- C45: Link https://www.mouser.pl/en/ProductDetail/Taiwan-Semiconductor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 -> (none)
- renumbered C23 to TP4
Connections:
- net HEATER_VOLTAGE_SENSE: now also C45.1
- net Masa: now also C45.2
